Commit message: Setup ros2_control and got the thrusters moving

File: urdf/auv.urdf.xacro (robot description, xacro)
@@ -1,10 +1,8 @@
 <?xml version="1.0"?>
 <robot xmlns:xacro="http://www.ros.org/wiki/xacro" name="auv">
-    <!-- <xacro:include filename="$(find calypso_sim)/urdf/camera2d.urdf.xacro"/> -->
-    <xacro:include filename="$(find calypso_sim)/urdf/camera_depth.urdf.xacro"/>
-    <xacro:include filename="$(find calypso_sim)/urdf/imu.urdf.xacro"/>
-    <xacro:include filename="$(find calypso_sim)/urdf/thrusters.urdf.xacro"/>
-    <xacro:include filename="$(find calypso_sim)/urdf/chasis.urdf.xacro"/>
-    <xacro:include filename="$(find calypso_sim)/urdf/dvl_snippets.urdf.xacro"/>
+    <xacro:arg name="controller_config_path" default="/tmp/placeholder.yaml"/>
+    <xacro:include filename="thrusters.urdf.xacro"/>
+    <xacro:include filename="chasis.urdf.xacro"/>
+    <xacro:include filename="ros2_control.urdf.xacro"/>
     <material name="red">
         <color rgba="1 0 0 1"/>
@@ -51,37 +49,9 @@
     <xacro:thruster_CCW id="8" parent="base_link" xyz="-0.45 0.2 0" rpy="0 1.57 0.785398" axis="0 0 -1">
     </xacro:thruster_CCW>
-    <xacro:default_dvl namespace="calypso_sim" parent_link="base_link">
+    <xacro:ros2_control_block controller_config_path="$(arg controller_config_path)"/>
+    <!-- <xacro:default_dvl namespace="calypso_sim" parent_link="base_link">
       <origin xyz="0 0 -0.18" rpy="0 0 0"/>
-    </xacro:default_dvl>
-    <xacro:imu id="1" parent="base_link" xyz="0 0 0" rpy="0 0 0"></xacro:imu>
-    <xacro:depth_cam id="1" parent="base_link" xyz="0.3 0 0" rpy="0 0 0"></xacro:depth_cam>
-    <gazebo>
-      <plugin name="gazebo_ros_control" filename="libgazebo_ros_control.so">
-          <!-- <robotNameSpace>/Kwad</robotNameSpace> -->
-          <robotSimType>gazebo_ros_control/DefaultRobotHWSim</robotSimType>
-      </plugin>
-    </gazebo>
-    <gazebo>
-      <plugin name="freebuoyancy_gazebo" filename="libfreebuoyancy_gazebo.so">
-        <descriptionParam>/robot_description</descriptionParam>
-        <alwaysOn>true</alwaysOn>
-        <surface>0 0 40</surface>
-        <updateRate>.001</updateRate>
-        <link name='base_link'>
-          <buoyancy>
-            <compensation>0.0</compensation>
-            <origin xyz="0 0 0"/>
-          </buoyancy>
-        </link>
-      </plugin>
-    </gazebo>
-  <!-- <gazebo>
-    <plugin name="BuoyancyPlugin" filename="libBuoyancyPlugin.so">
-    <fluid_density>1200</fluid_density>
-    <link name="base_link">
-      <volume>240</volume>
-      <center_of_volume>0 0 0</center_of_volume>
-    </link>
-  </plugin>
-</gazebo> -->
+    </xacro:default_dvl> -->
+    <!-- <xacro:imu id="1" parent="base_link" xyz="0 0 0" rpy="0 0 0"></xacro:imu> -->
+    <!-- <xacro:depth_cam id="1" parent="base_link" xyz="0.3 0 0" rpy="0 0 0"></xacro:depth_cam> -->
 </robot>

File: urdf/chasis.urdf.xacro (robot description, xacro)
@@ -21,74 +21,8 @@
     </inertial> -->
     <inertial>
-      <mass value="42.775"/>
+      <mass value="42000.775"/>
       <inertia ixx="0" ixy="0" ixz="0" iyy="0" iyz="0" izz="0"/>
     </inertial>
   </link>
-  <!-- <link name="right_leg">
-    <visual>
-      <geometry>
-        <box size="0.6 0.1 0.2"/>
-      </geometry>
-      <material name="red"/>
-    </visual>
-    <collision>
-      <geometry>
-          <box size="0.6 0.1 0.2"/>
-      </geometry>
-    </collision>
-    <inertial>
-      <mass value="1"/>
-      <inertia ixx="0" ixy="0" ixz="0" iyy="0" iyz="0" izz="0"/>
-    </inertial>
-  </link>
-  <joint name="base_to_right_leg" type="fixed">
-    <parent link="base_link"/>
-    <child link="right_leg"/>
-    <origin xyz="0 -0.22 -0.1"/>
-  </joint> -->
-  <!-- <link name="left_leg">
-    <visual>
-      <geometry>
-        <box size="0.6 0.1 0.2"/>
-      </geometry>
-      <material name="red"/>
-    </visual>
-    <collision>
-      <geometry>
-        <box size="0.6 0.1 0.2"/>
-      </geometry>
-    </collision>
-    <inertial>
-      <mass value="1"/>
-      <inertia ixx="0" ixy="0.0" ixz="0.0" iyy="0" iyz="0.0" izz="0"/>
-    </inertial>
-  </link>
-  <joint name="base_to_left_leg" type="fixed">
-    <parent link="base_link"/>
-    <child link="left_leg"/>
-    <origin xyz="0 0.22 -0.1"/>
-  </joint> -->
-    <!-- <link name="head">
-      <visual>
-        <geometry>
-          <sphere radius="0.2"/>
-        </geometry>
-        <material name="green"/>
-      </visual>
-      <collision>
-        <geometry>
-          <sphere radius="0.2"/>
-        </geometry>
-      </collision>
-      <inertial>
-        <mass value="0.1"/>
-      <inertia ixx="0" ixy="0.0" ixz="0.0" iyy="0" iyz="0.0" izz="0"/>
-    </inertial>
-    </link>
- <joint name="head_to_base" type="fixed">
-    <parent link="base_link"/>
-    <child link="head"/>
-    <origin rpy="0 0 0" xyz="0.3 0 0"/>
-  </joint> -->
   </xacro:macro>
 </robot>

File: urdf/thrusters.urdf.xacro (robot description, xacro)
@@ -1,6 +1,6 @@
 <?xml version='1.0'?>
 <robot xmlns:xacro="http://www.ros.org/wiki/xacro" name="thruster">
-  <xacro:property name="thrusterCCW_path" value="package://calypso_sim/meshes/thrusters/T200_Thruster_CCW/meshes/"/>
-  <xacro:property name="thrusterCW_path" value="package://calypso_sim/meshes/thrusters/T200_Thruster_CW/meshes/"/>
+  <xacro:property name="thrusterCCW_path" value="file://$(find calypso2)/meshes/thrusters/T200_Thruster_CCW/meshes/"/>
+  <xacro:property name="thrusterCW_path" value="file://$(find calypso2)/meshes/thrusters/T200_Thruster_CW/meshes/"/>
    <xacro:macro name="thruster_CCW" params="id parent xyz rpy axis">
     <link name="thruster_${id}_link">
@@ -48,16 +48,16 @@
       <axis xyz="${axis}"/>
     </joint>
-    <transmission name="thruster_${id}_trainsmission" >
+    <!-- <transmission name="thruster_${id}_trainsmission" >
       <type>transmission_interface/SimpleTransmission</type>
         <joint name="prop_${id}_to_thruster_${id}_joint">
           <hardwareInterface>hardware_interface/VelocityJointInterface</hardwareInterface>
         </joint>
-      <actuator name="BLDC_motor_${id}">
+      <actuator name="thruster_${id}_motor">
         <hardwareInterface>hardware_interface/VelocityJointInterface</hardwareInterface>
         <mechanicalReduction>1</mechanicalReduction>
       </actuator>
-	  </transmission>
+	  </transmission> -->
     <gazebo>
-      <plugin name='blade_1_${id}' filename='libLiftDragPlugin.so'>
+      <plugin filename="ignition-gazebo-lift-drag-system" name="ignition::gazebo::systems::LiftDrag">
         <a0>0.3</a0>
         <alpha_stall>1.4</alpha_stall>
@@ -75,5 +75,5 @@
         <link_name>prop_${id}</link_name>
       </plugin>
-      <plugin name='blade_2_${id}' filename='libLiftDragPlugin.so'>
+      <plugin filename="ignition-gazebo-lift-drag-system" name="ignition::gazebo::systems::LiftDrag">
         <a0>0.3</a0>
         <alpha_stall>1.4</alpha_stall>
@@ -95,18 +95,4 @@
       <static>0</static>
       <allow_auto_disable>0</allow_auto_disable>
-    </gazebo>
-    <!-- <gazebo>
-      <plugin name="freefloating_gazebo_control" filename="libfreefloating_gazebo_control.so">
-        <switchService>switch</switchService>
-        <updateRate>100</updateRate>
-        <link>base_link</link>
-        <thruster>
-            <map>${xyz} ${rpy}</map>
-            <effort>30</effort>
-        </thruster>
-      </plugin>
-    </gazebo> -->
-     <gazebo reference="prop_${id}">
-        <material>Gazebo/Red</material>
     </gazebo>
   </xacro:macro>
@@ -157,5 +143,5 @@
       <axis xyz="${axis}"/>
     </joint>
-    <transmission name="thruster_${id}_trainsmission" >
+    <!-- <transmission name="thruster_${id}_trainsmission" >
       <type>transmission_interface/SimpleTransmission</type>
         <joint name="prop_${id}_to_thruster_${id}_joint">
@@ -166,7 +152,7 @@
         <mechanicalReduction>1</mechanicalReduction>
       </actuator>
-	  </transmission>
+	  </transmission> -->
     <gazebo>
-      <plugin name='blade_1_${id}' filename='libLiftDragPlugin.so'>
+      <plugin filename="ignition-gazebo-lift-drag-system" name="ignition::gazebo::systems::LiftDrag">
         <a0>0.3</a0>
         <alpha_stall>1.4</alpha_stall>
@@ -184,5 +170,5 @@
         <link_name>prop_${id}</link_name>
       </plugin>
-      <plugin name='blade_2_${id}' filename='libLiftDragPlugin.so'>
+      <plugin filename="ignition-gazebo-lift-drag-system" name="ignition::gazebo::systems::LiftDrag">
         <a0>0.3</a0>
         <alpha_stall>1.4</alpha_stall>
@@ -205,18 +191,4 @@
       <allow_auto_disable>0</allow_auto_disable>
     </gazebo>
-  <!-- <gazebo>
-      <plugin name="freefloating_gazebo_control" filename="libfreefloating_gazebo_control.so">
-        <switchService>switch</switchService>
-        <updateRate>100</updateRate>
-        <link>base_link</link>
-        <thruster>
-            <map>-1 0 0 0 0 ${-body_width/2}</map>
-            <effort>30</effort>
-        </thruster>
-      </plugin>
-  </gazebo> -->
-    <gazebo reference="prop_${id}">
-      <material>Gazebo/Green</material>
-    </gazebo>
   </xacro:macro>
 </robot>
